File: safe-basic.kicad_sch (KiCad schematic)
At the start: 1 part

Commit message: test: change resistor value for BoardReadyOps E2E
Parts:
- R1: value 10k -> 12k
Changed lines of the file:
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@@
     (lib_id "Device:R")
     (property "Reference" "R1")
-    (property "Value" "10k")
+    (property "Value" "12k")
     (property "Footprint" "Resistor_SMD:R_0603")
     (property "Manufacturer" "Yageo")

Commit message: test: update resistor value to 15k for E2E validation
Parts:
- R1: value 12k -> 15k; MPN RC0603FR-0710KL -> RC0603FR-0715KL
Changed lines of the file:
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@@
     (lib_id "Device:R")
     (property "Reference" "R1")
-    (property "Value" "12k")
+    (property "Value" "15k")
     (property "Footprint" "Resistor_SMD:R_0603")
     (property "Manufacturer" "Yageo")
-    (property "MPN" "RC0603FR-0710KL")
+    (property "MPN" "RC0603FR-0715KL")
   )
   (label "MCU_PA0")
